File: PCB/RfLink-ESPlink.sch (EAGLE design)
At the start: 54 parts, among them IC1 WEMOS D1 MINI, IC2 ARDUINO-MEGA, IC3 PRO MINI 3.3V, IC4 CC2500 MODUL, IC5 TRANSMITTER 433MHZ, IC6 RXB6, IC7 RTX-MID, IC8 NRF24L01A, J2 JUMPER-3SMD, U1 AMS1117, U2 DHT22, U3 DS18B20, X1 BU-SMA-V

Commit message: Update Schema
Moved R5 closer to Mega 2560
Connections:
- net RX-TX renamed ESP-TX
- net TX-RX-L renamed ESP-RX
Other:
- moved on the sheet: R5
Changed lines of the file:
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@@
 </instance>
 <instance part="JP2" gate="G$1" x="325.12" y="182.88" rot="R180"/>
-<instance part="R5" gate="G$1" x="243.84" y="172.72" smashed="yes">
-<attribute name="NAME" x="240.03" y="169.1386" size="1.778" layer="95"/>
-<attribute name="VALUE" x="245.11" y="169.418" size="1.778" layer="96"/>
+<instance part="R5" gate="G$1" x="33.02" y="154.94" smashed="yes">
+<attribute name="NAME" x="29.21" y="151.3586" size="1.778" layer="95"/>
+<attribute name="VALUE" x="34.29" y="151.638" size="1.778" layer="96"/>
 </instance>
 <instance part="U$13" gate="G$1" x="25.4" y="137.16" smashed="yes">
@@
 <segment>
 <pinref part="IC1" gate="D1" pin="3V3"/>
-<wire x1="195.58" y1="157.48" x2="182.88" y2="157.48" width="0.1524" layer="91"/>
-<label x="182.88" y="157.48" size="1.778" layer="95"/>
+<wire x1="195.58" y1="157.48" x2="180.34" y2="157.48" width="0.1524" layer="91"/>
+<label x="180.34" y="157.48" size="1.778" layer="95"/>
 </segment>
 <segment>
@@
 </segment>
 </net>
-<net name="RX-TX" class="0">
+<net name="ESP-TX" class="0">
 <segment>
 <pinref part="IC2" gate="G$1" pin="0(RX0)"/>
-<wire x1="43.18" y1="157.48" x2="25.4" y2="157.48" width="0.1524" layer="91"/>
-<label x="30.48" y="157.48" size="1.778" layer="95"/>
-</segment>
-<segment>
-<label x="251.46" y="175.26" size="1.778" layer="95"/>
+<wire x1="43.18" y1="157.48" x2="22.86" y2="157.48" width="0.1524" layer="91"/>
+<label x="22.86" y="157.48" size="1.778" layer="95" rot="MR0"/>
+</segment>
+<segment>
+<label x="236.22" y="175.26" size="1.778" layer="95"/>
 <pinref part="IC1" gate="D1" pin="TX"/>
-<wire x1="228.6" y1="175.26" x2="256.54" y2="175.26" width="0.1524" layer="91"/>
+<wire x1="228.6" y1="175.26" x2="236.22" y2="175.26" width="0.1524" layer="91"/>
 </segment>
 <segment>
@@
 <segment>
 <pinref part="IC2" gate="G$1" pin="1(TX0)"/>
-<wire x1="43.18" y1="154.94" x2="25.4" y2="154.94" width="0.1524" layer="91"/>
-<label x="30.48" y="154.94" size="1.778" layer="95"/>
-</segment>
-<segment>
+<wire x1="43.18" y1="154.94" x2="38.1" y2="154.94" width="0.1524" layer="91"/>
+<label x="38.1" y="154.94" size="1.778" layer="95"/>
 <pinref part="R5" gate="G$1" pin="2"/>
-<wire x1="248.92" y1="172.72" x2="256.54" y2="172.72" width="0.1524" layer="91"/>
-<label x="251.46" y="172.72" size="1.778" layer="95"/>
-</segment>
-</net>
-<net name="TX-RX-L" class="0">
-<segment>
-<pinref part="R5" gate="G$1" pin="1"/>
+</segment>
+</net>
+<net name="ESP-RX" class="0">
+<segment>
 <pinref part="IC1" gate="D1" pin="RX"/>
-<wire x1="238.76" y1="172.72" x2="228.6" y2="172.72" width="0.1524" layer="91"/>
-<label x="228.6" y="172.72" size="1.778" layer="95"/>
+<wire x1="236.22" y1="172.72" x2="228.6" y2="172.72" width="0.1524" layer="91"/>
+<label x="236.22" y="172.72" size="1.778" layer="95"/>
 </segment>
 <segment>
@@
 <pinref part="LED1" gate="G$1" pin="C"/>
 <wire x1="233.68" y1="101.6" x2="233.68" y2="104.14" width="0.1524" layer="91"/>
+</segment>
+<segment>
+<pinref part="R5" gate="G$1" pin="1"/>
+<wire x1="27.94" y1="154.94" x2="22.86" y2="154.94" width="0.1524" layer="91"/>
+<label x="22.86" y="154.94" size="1.778" layer="95" rot="R180"/>
 </segment>
 </net>
@@
 <segment>
 <pinref part="IC1" gate="D1" pin="D3"/>
-<wire x1="228.6" y1="165.1" x2="238.76" y2="165.1" width="0.1524" layer="91"/>
-<label x="231.14" y="165.1" size="1.778" layer="95"/>
+<wire x1="228.6" y1="165.1" x2="236.22" y2="165.1" width="0.1524" layer="91"/>
+<label x="236.22" y="165.1" size="1.778" layer="95"/>
 </segment>
 <segment>
@@
 <segment>
 <pinref part="IC1" gate="D1" pin="D4"/>
-<wire x1="228.6" y1="162.56" x2="238.76" y2="162.56" width="0.1524" layer="91"/>
-<label x="231.14" y="162.56" size="1.778" layer="95"/>
+<wire x1="228.6" y1="162.56" x2="236.22" y2="162.56" width="0.1524" layer="91"/>
+<label x="236.22" y="162.56" size="1.778" layer="95"/>
 </segment>
 </net>
@@
 <segment>
 <pinref part="IC1" gate="D1" pin="D6"/>
-<wire x1="195.58" y1="165.1" x2="182.88" y2="165.1" width="0.1524" layer="91"/>
-<label x="182.88" y="165.1" size="1.778" layer="95"/>
+<wire x1="195.58" y1="165.1" x2="180.34" y2="165.1" width="0.1524" layer="91"/>
+<label x="180.34" y="165.1" size="1.778" layer="95"/>
 </segment>
 <segment>
@@
 <segment>
 <pinref part="IC1" gate="D1" pin="A0"/>
-<wire x1="195.58" y1="172.72" x2="182.88" y2="172.72" width="0.1524" layer="91"/>
-<label x="182.88" y="172.72" size="1.778" layer="95"/>
+<wire x1="195.58" y1="172.72" x2="180.34" y2="172.72" width="0.1524" layer="91"/>
+<label x="180.34" y="172.72" size="1.778" layer="95"/>
 </segment>
 <segment>
@@
 <segment>
 <pinref part="IC1" gate="D1" pin="D5"/>
-<wire x1="195.58" y1="167.64" x2="182.88" y2="167.64" width="0.1524" layer="91"/>
-<label x="182.88" y="167.64" size="1.778" layer="95"/>
+<wire x1="195.58" y1="167.64" x2="180.34" y2="167.64" width="0.1524" layer="91"/>
+<label x="180.34" y="167.64" size="1.778" layer="95"/>
 </segment>
 </net>
@@
 <segment>
 <pinref part="IC1" gate="D1" pin="D0"/>
-<wire x1="195.58" y1="170.18" x2="180.34" y2="170.18" width="0.1524" layer="91"/>
+<wire x1="195.58" y1="170.18" x2="193.04" y2="170.18" width="0.1524" layer="91"/>
 <pinref part="D0" gate="1" pin="P"/>
-<wire x1="195.58" y1="170.18" x2="195.58" y2="147.32" width="0.1524" layer="91"/>
+<wire x1="193.04" y1="170.18" x2="180.34" y2="170.18" width="0.1524" layer="91"/>
 <pinref part="R9" gate="G$1" pin="2"/>
-<wire x1="195.58" y1="147.32" x2="254" y2="147.32" width="0.1524" layer="91"/>
-<wire x1="254" y1="147.32" x2="254" y2="121.92" width="0.1524" layer="91"/>
-<junction x="195.58" y="170.18"/>
+<wire x1="193.04" y1="144.78" x2="254" y2="144.78" width="0.1524" layer="91"/>
+<wire x1="254" y1="144.78" x2="254" y2="121.92" width="0.1524" layer="91"/>
+<wire x1="193.04" y1="144.78" x2="193.04" y2="170.18" width="0.1524" layer="91"/>
+<junction x="193.04" y="170.18"/>
 </segment>
 </net>
@@
 <segment>
 <pinref part="IC1" gate="D1" pin="D7"/>
-<wire x1="195.58" y1="162.56" x2="182.88" y2="162.56" width="0.1524" layer="91"/>
-<label x="182.88" y="162.56" size="1.778" layer="95"/>
+<wire x1="195.58" y1="162.56" x2="180.34" y2="162.56" width="0.1524" layer="91"/>
+<label x="180.34" y="162.56" size="1.778" layer="95"/>
 </segment>
 </net>
@@
 <wire x1="180.34" y1="160.02" x2="190.5" y2="160.02" width="0.1524" layer="91"/>
 <wire x1="190.5" y1="160.02" x2="195.58" y2="160.02" width="0.1524" layer="91"/>
-<wire x1="190.5" y1="160.02" x2="190.5" y2="144.78" width="0.1524" layer="91"/>
+<wire x1="190.5" y1="160.02" x2="190.5" y2="139.7" width="0.1524" layer="91"/>
 <pinref part="R8" gate="G$1" pin="2"/>
-<wire x1="190.5" y1="144.78" x2="246.38" y2="144.78" width="0.1524" layer="91"/>
-<wire x1="246.38" y1="144.78" x2="246.38" y2="121.92" width="0.1524" layer="91"/>
+<wire x1="190.5" y1="139.7" x2="246.38" y2="139.7" width="0.1524" layer="91"/>
+<wire x1="246.38" y1="139.7" x2="246.38" y2="121.92" width="0.1524" layer="91"/>
 <junction x="190.5" y="160.02"/>
 </segment>
@@
 <segment>
 <pinref part="IC1" gate="D1" pin="5V"/>
-<wire x1="256.54" y1="157.48" x2="228.6" y2="157.48" width="0.1524" layer="91"/>
+<wire x1="251.46" y1="157.48" x2="228.6" y2="157.48" width="0.1524" layer="91"/>
 <label x="251.46" y="157.48" size="1.778" layer="95"/>
 </segment>

Commit message: New pcb revison 0.81
Added resistors to all Arduino Mega 2560 pins connected to ESP, value
470R. Added JP5 for external power supplt if Mega not are in use.
Unnecessary pins removed from Mega 2560.
Parts:
- removed R26: 4k7, kb20:RESISTORR0805
- added JP5: (no value), kb20:GS015S-3.81-2P
- added R10, R11: 1K, kb20:RESISTORR0805
- IC2: value ARDUINO-MEGA -> ARDUINO MEGA 2560; device SparkFun:ARDUINO-MEGA -> SparkFun:ARDUINO-MEGA-MINI
- R1, R2, R3, R4, R5, R6: value 1K -> 470R
- R7: value 1k -> 470R
- R9: value 1K -> 1k
Connections:
- removed net GPIO12: IC1.D6, IC2.RESET, IC3.RST@2
- removed net TX-RX: IC2.1(TX0), R5.2
- new net GPIO12-RESET: IC1.D6, IC3.RST@2, R1.2
- new net MEGA-RX: IC2.0(RX0), R2.1
- new net MEGA-TX: IC2.1(TX0), R3.2
- new net RESET: IC2.RESET, R1.1
- net +3V3: now also R21.2, R23.2, R9.2; no longer R22.2, R24.2, R7.2
- net A0: now also R25.2; no longer R26.2
- net D3-GPIO0: no longer R21.2
- net ESP-RX: now also R3.1; no longer R5.1
- net ESP-TX: now also R2.2; no longer IC2.0(RX0)
- net GND: now also JP5.2, R22.1, R24.1, R8.1; no longer R21.1, R23.1, R26.1, R6.1
- net GPIO13-D7: now also R21.1, R22.2; no longer R22.1, R23.2
- net GPIO14-D5: now also R23.1, R24.2; no longer R24.1, R25.2
- net MEGA5V: now also JP5.1
- net N$1: now also R4.1; no longer R1.1
- net N$11: now also R7.2; no longer R3.2
- net N$12: now also R5.2; no longer R4.2
- net N$13: now also R4.2; no longer R1.2
- net N$16: now also R9.1; no longer R7.1
- net N$17: now also R10.1; no longer R8.1
- net N$18: now also R8.2; no longer R6.2
- net N$19: now also R11.2; no longer R9.2
- net N$2: now also R5.1; no longer R4.1
- net N$3: now also R6.1; no longer R2.1
- net N$4: now also R7.1; no longer R3.1
- net N$7: now also R11.1; no longer R9.1
- net N$8: now also R10.2; no longer R8.2
- net N$9: now also R6.2; no longer R2.2
Other:
- note added: "0.81"
- note added: "Ext power"
- moved on the sheet: C1, PS2, R1, R2, R21, R22, R23, R24, R25, R3, R4, R5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

Commit message: New pcb revison 0.9
Added ESP-01 for easy serial debug of Wemos ESP. This is the
manufactured version. And some other good to have functions!
Parts:
- added +3.3V, P1, P10, P11, P12, P13, P14, P15, P16, P17, P18, P19, P2, P20, P21, P22, P23, P24, P25, P3, P4, P5, P6, P7, P8, P9: (no value), wirepad:1,6/0,9
- added C9: 10μF, rcl:CPOL-EUE2-5
- added D6: D6, wirepad:1,6/0,9
- added GND5, GND7: GND, wirepad:1,6/0,9
- added GPIO2: IO2, wirepad:1,6/0,9
- added IC9: ESP-01, esp8266modules:ESP01
- added R12, R13: 4k7, kb20:RESISTORR0805
- added RX: RX, wirepad:1,6/0,9
- added TX: TX, wirepad:1,6/0,9
Connections:
- new net ESP-RESET: IC1.RESET, IC9.GPIO0
- new net N$24: IC9.CH_PD, R12.1
- new net N$26: IC9.RST, R13.1
- new net N$27: GPIO2.P, IC9.GPIO2
- new net N$28: P1.P, P2.P, P3.P, P4.P, P5.P
- new net N$29: P10.P, P6.P, P7.P, P8.P, P9.P
- new net N$31: P16.P, P17.P, P18.P, P19.P, P20.P
- net +3V3: now also +3.3V.P, C9.+, IC9.VCC, P21.P, P22.P, P23.P, P24.P, P25.P, R12.2, R13.2
- net ESP-RX: now also IC9.TXD, RX.P
- net ESP-TX: now also IC9.RXD, TX.P
- net GND: now also C9.-, GND5.P, GND7.P, IC9.GND, P11.P, P12.P, P13.P, P14.P, P15.P
- net GPIO14-D5: now also D6.P
Other:
- note added: "0.9"
- note added: "Debug Option"
- note removed: "0.81"
- moved on the sheet: C1, C2, C3, C4, D0, D8, JP5, PS1, PS2, U1, VCC1, VCC2
